File: PROJECTS/TUTORIALS/BlinkyBoard/v1.brd (EAGLE design)
At the start: 25.1 x 30.5 mm, 10 parts, among them IC1 LM555D

Commit message: update
finished tutorial 02
Parts:
- moved C1 3.23 mm to (7.16, 25.5), turned to 90 degrees
- moved R2 2.47 mm to (3.21, 20.5)
- moved C2 1.90 mm to (3.28, 26.1), turned to 90 degrees
- moved LED1 0.85 mm to (19.6, 26.1)
- moved LED2 0.85 mm to (19.6, 19.6)
- moved R1 0.60 mm to (3.21, 15.2)
Routing:
- net VCC: track 0.00 -> 47.3 mm
- net N$6: track 0.00 -> 20.1 mm, vias 0 -> 2
- net N$2: track 0.00 -> 8.41 mm
- net N$5: track 0.00 -> 7.27 mm
- net N$1: track 0.00 -> 4.63 mm
- net N$3: track 0.00 -> 4.05 mm
- net N$7: track 0.00 -> 3.45 mm
Other:
- board size 25.1 x 30.5 mm -> 25.1 x 32.3 mm
- board text added: "Blinker v1"
