File: PROJECTS/IDers Test/SMM Test Jig/LPC_probe.brd (EAGLE design)
At the start: 17.8 x 35.2 mm, 2 parts, among them X1 1365-10, X2 1365-10

Commit message: update
Routing:
- net N$10: track 44.7 -> 16.9 mm
- net N$1: track 43.7 -> 16.8 mm
- net N$6: track 16.4 -> 40.9 mm
- net N$5: track 18.7 -> 40.8 mm
- net N$9: track 38.2 -> 17.0 mm
- net N$2: track 36.5 -> 29.6 mm
- net N$7: track 16.9 -> 19.5 mm
- net N$3: track 19.7 -> 18.3 mm
