File: PROJECTS/IDers Test/SMM Test Jig/CPLD_probe.brd (EAGLE design)
At the start: 24.1 x 40.3 mm, 2 parts

Commit message: update
Routing:
- net N$3: track 23.9 -> 38.0 mm
- net N$2: track 37.0 -> 28.2 mm
- net N$1: track 29.1 -> 33.3 mm
- net N$5: track 22.3 -> 24.7 mm
- net N$6: track 17.4 -> 18.8 mm
- net N$4: track 20.7 -> 19.9 mm
Changed lines of the file:
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@@
 </class>
 </classes>
-<designrules name="default">
+<designrules name="default *">
 <description language="de">&lt;b&gt;EAGLE Design Rules&lt;/b&gt;
 &lt;p&gt;
@@
 <param name="mtCopper" value="0.035mm 0.035mm 0.035mm 0.035mm 0.035mm 0.035mm 0.035mm 0.035mm 0.035mm 0.035mm 0.035mm 0.035mm 0.035mm 0.035mm 0.035mm 0.035mm"/>
 <param name="mtIsolate" value="1.5mm 0.15mm 0.2mm 0.15mm 0.2mm 0.15mm 0.2mm 0.15mm 0.2mm 0.15mm 0.2mm 0.15mm 0.2mm 0.15mm 0.2mm"/>
-<param name="mdWireWire" value="8mil"/>
-<param name="mdWirePad" value="8mil"/>
-<param name="mdWireVia" value="8mil"/>
-<param name="mdPadPad" value="8mil"/>
-<param name="mdPadVia" value="8mil"/>
-<param name="mdViaVia" value="8mil"/>
-<param name="mdSmdPad" value="8mil"/>
-<param name="mdSmdVia" value="8mil"/>
-<param name="mdSmdSmd" value="8mil"/>
+<param name="mdWireWire" value="14mil"/>
+<param name="mdWirePad" value="14mil"/>
+<param name="mdWireVia" value="14mil"/>
+<param name="mdPadPad" value="14mil"/>
+<param name="mdPadVia" value="14mil"/>
+<param name="mdViaVia" value="14mil"/>
+<param name="mdSmdPad" value="14mil"/>
+<param name="mdSmdVia" value="14mil"/>
+<param name="mdSmdSmd" value="14mil"/>
 <param name="mdViaViaSameLayer" value="8mil"/>
 <param name="mnLayersViaInSmd" value="2"/>
@@
 <param name="mdDrill" value="8mil"/>
 <param name="mdSmdStop" value="0mil"/>
-<param name="msWidth" value="10mil"/>
-<param name="msDrill" value="24mil"/>
+<param name="msWidth" value="14mil"/>
+<param name="msDrill" value="26mil"/>
 <param name="msMicroVia" value="9.99mm"/>
 <param name="msBlindViaRatio" value="0.5"/>
@@
 <param name="RoutingGrid" value="50mil"/>
 <param name="AutoGrid" value="1"/>
-<param name="Efforts" value="1"/>
+<param name="Efforts" value="2"/>
 <param name="TopRouterVariant" value="1"/>
 <param name="tpViaShape" value="round"/>
-<param name="PrefDir.1" value="-"/>
+<param name="PrefDir.1" value="a"/>
 <param name="PrefDir.2" value="0"/>
 <param name="PrefDir.3" value="0"/>
@@
 <contactref element="SV2" pad="2"/>
 <contactref element="SV1" pad="2"/>
-<wire x1="8.4328" y1="16.002" x2="5.2324" y2="12.8016" width="0.254" layer="1"/>
-<wire x1="8.4328" y1="31.3182" x2="8.4328" y2="16.002" width="0.254" layer="1"/>
-<wire x1="11.8618" y1="34.7472" x2="8.4328" y2="31.3182" width="0.254" layer="1"/>
-<wire x1="13.6906" y1="34.7472" x2="11.8618" y2="34.7472" width="0.254" layer="1"/>
-<wire x1="15.2908" y1="33.147" x2="13.6906" y2="34.7472" width="0.254" layer="1"/>
-<wire x1="5.2324" y1="12.8016" x2="5.08" y2="12.7" width="0.254" layer="1"/>
-<wire x1="15.2908" y1="33.147" x2="15.24" y2="33.02" width="0.254" layer="1"/>
+<wire x1="5.08" y1="12.7" x2="5.08" y2="31.75" width="0.4064" layer="1"/>
+<wire x1="5.08" y1="31.75" x2="8.89" y2="35.56" width="0.4064" layer="1"/>
+<wire x1="8.89" y1="35.56" x2="15.24" y2="35.56" width="0.4064" layer="1"/>
+<wire x1="15.24" y1="35.56" x2="15.24" y2="33.02" width="0.4064" layer="1"/>
 </signal>
 <signal name="N$2">
 <contactref element="SV2" pad="1"/>
 <contactref element="SV1" pad="1"/>
-<wire x1="5.2324" y1="9.8298" x2="5.2324" y2="10.0584" width="0.254" layer="1"/>
-<wire x1="6.604" y1="8.4582" x2="5.2324" y2="9.8298" width="0.254" layer="1"/>
-<wire x1="10.9474" y1="8.4582" x2="6.604" y2="8.4582" width="0.254" layer="1"/>
-<wire x1="17.1196" y1="14.6304" x2="10.9474" y2="8.4582" width="0.254" layer="1"/>
-<wire x1="17.1196" y1="30.1752" x2="17.1196" y2="14.6304" width="0.254" layer="1"/>
-<wire x1="15.5194" y1="31.7754" x2="17.1196" y2="30.1752" width="0.254" layer="1"/>
-<wire x1="14.8336" y1="31.7754" x2="15.5194" y2="31.7754" width="0.254" layer="1"/>
-<wire x1="14.3764" y1="32.2326" x2="14.8336" y2="31.7754" width="0.254" layer="1"/>
-<wire x1="13.9192" y1="31.7754" x2="14.3764" y2="32.2326" width="0.254" layer="1"/>
-<wire x1="12.7762" y1="32.9184" x2="13.9192" y2="31.7754" width="0.254" layer="1"/>
-<wire x1="5.2324" y1="10.0584" x2="5.08" y2="10.16" width="0.254" layer="1"/>
-<wire x1="12.7762" y1="32.9184" x2="12.7" y2="33.02" width="0.254" layer="1"/>
+<wire x1="5.08" y1="10.16" x2="6.35" y2="11.43" width="0.4064" layer="1"/>
+<wire x1="6.35" y1="11.43" x2="6.35" y2="30.48" width="0.4064" layer="1"/>
+<wire x1="6.35" y1="30.48" x2="8.89" y2="33.02" width="0.4064" layer="1"/>
+<wire x1="8.89" y1="33.02" x2="12.7" y2="33.02" width="0.4064" layer="1"/>
 </signal>
 <signal name="N$3">
 <contactref element="SV2" pad="3"/>
 <contactref element="SV1" pad="3"/>
-<wire x1="5.9182" y1="11.8872" x2="7.5184" y2="10.287" width="0.254" layer="1"/>
-<wire x1="6.3754" y1="12.3444" x2="5.9182" y2="11.8872" width="0.254" layer="1"/>
-<wire x1="6.3754" y1="13.0302" x2="6.3754" y2="12.3444" width="0.254" layer="1"/>
-<wire x1="8.89" y1="15.5448" x2="6.3754" y2="13.0302" width="0.254" layer="1"/>
-<wire x1="8.89" y1="26.7462" x2="8.89" y2="15.5448" width="0.254" layer="1"/>
-<wire x1="12.5476" y1="30.4038" x2="8.89" y2="26.7462" width="0.254" layer="1"/>
-<wire x1="7.5184" y1="10.287" x2="7.62" y2="10.16" width="0.254" layer="1"/>
-<wire x1="12.5476" y1="30.4038" x2="12.7" y2="30.48" width="0.254" layer="1"/>
+<wire x1="7.62" y1="10.16" x2="10.16" y2="7.62" width="0.4064" layer="1"/>
+<wire x1="10.16" y1="7.62" x2="12.7" y2="7.62" width="0.4064" layer="1"/>
+<wire x1="12.7" y1="7.62" x2="17.78" y2="12.7" width="0.4064" layer="1"/>
+<wire x1="17.78" y1="12.7" x2="17.78" y2="31.75" width="0.4064" layer="1"/>
+<wire x1="17.78" y1="31.75" x2="13.97" y2="31.75" width="0.4064" layer="1"/>
+<wire x1="13.97" y1="31.75" x2="12.7" y2="30.48" width="0.4064" layer="1"/>
 </signal>
 <signal name="N$4">
 <contactref element="SV2" pad="5"/>
 <contactref element="SV1" pad="5"/>
-<wire x1="8.4328" y1="11.8872" x2="10.16" y2="10.16" width="0.254" layer="1"/>
-<wire x1="8.89" y1="12.3444" x2="8.4328" y2="11.8872" width="0.254" layer="1"/>
-<wire x1="8.89" y1="13.0302" x2="8.89" y2="12.3444" width="0.254" layer="1"/>
-<wire x1="8.4328" y1="13.4874" x2="8.89" y2="13.0302" width="0.254" layer="1"/>
-<wire x1="8.4328" y1="13.716" x2="8.4328" y2="13.4874" width="0.254" layer="1"/>
-<wire x1="9.8044" y1="15.0876" x2="8.4328" y2="13.716" width="0.254" layer="1"/>
-<wire x1="9.8044" y1="25.146" x2="9.8044" y2="15.0876" width="0.254" layer="1"/>
-<wire x1="12.5476" y1="27.8892" x2="9.8044" y2="25.146" width="0.254" layer="1"/>
-<wire x1="12.5476" y1="27.8892" x2="12.7" y2="27.94" width="0.254" layer="1"/>
+<wire x1="10.16" y1="10.16" x2="8.89" y2="11.43" width="0.4064" layer="1"/>
+<wire x1="8.89" y1="11.43" x2="8.89" y2="13.97" width="0.4064" layer="1"/>
+<wire x1="8.89" y1="13.97" x2="12.7" y2="17.78" width="0.4064" layer="1"/>
+<wire x1="12.7" y1="17.78" x2="12.7" y2="27.94" width="0.4064" layer="1"/>
 </signal>
 <signal name="N$5">
 <contactref element="SV2" pad="4"/>
 <contactref element="SV1" pad="4"/>
-<wire x1="7.5184" y1="13.4874" x2="7.5184" y2="12.8016" width="0.254" layer="1"/>
-<wire x1="9.3472" y1="15.3162" x2="7.5184" y2="13.4874" width="0.254" layer="1"/>
-<wire x1="9.3472" y1="26.289" x2="9.3472" y2="15.3162" width="0.254" layer="1"/>
-<wire x1="12.0904" y1="29.0322" x2="9.3472" y2="26.289" width="0.254" layer="1"/>
-<wire x1="13.2334" y1="29.0322" x2="12.0904" y2="29.0322" width="0.254" layer="1"/>
-<wire x1="13.462" y1="28.8036" x2="13.2334" y2="29.0322" width="0.254" layer="1"/>
-<wire x1="13.6906" y1="28.8036" x2="13.462" y2="28.8036" width="0.254" layer="1"/>
-<wire x1="13.9192" y1="29.0322" x2="13.6906" y2="28.8036" width="0.254" layer="1"/>
-<wire x1="13.9192" y1="29.2608" x2="13.9192" y2="29.0322" width="0.254" layer="1"/>
-<wire x1="15.0622" y1="30.4038" x2="13.9192" y2="29.2608" width="0.254" layer="1"/>
-<wire x1="7.5184" y1="12.8016" x2="7.62" y2="12.7" width="0.254" layer="1"/>
-<wire x1="15.0622" y1="30.4038" x2="15.24" y2="30.48" width="0.254" layer="1"/>
+<wire x1="7.62" y1="12.7" x2="7.62" y2="29.21" width="0.4064" layer="1"/>
+<wire x1="7.62" y1="29.21" x2="13.97" y2="29.21" width="0.4064" layer="1"/>
+<wire x1="13.97" y1="29.21" x2="15.24" y2="30.48" width="0.4064" layer="1"/>
 </signal>
 <signal name="N$6">
 <contactref element="SV2" pad="6"/>
 <contactref element="SV1" pad="6"/>
-<wire x1="10.2616" y1="23.0886" x2="10.2616" y2="12.8016" width="0.254" layer="1"/>
-<wire x1="15.0622" y1="27.8892" x2="10.2616" y2="23.0886" width="0.254" layer="1"/>
-<wire x1="10.2616" y1="12.8016" x2="10.16" y2="12.7" width="0.254" layer="1"/>
-<wire x1="15.0622" y1="27.8892" x2="15.24" y2="27.94" width="0.254" layer="1"/>
+<wire x1="15.24" y1="27.94" x2="15.24" y2="15.24" width="0.4064" layer="1"/>
+<wire x1="15.24" y1="15.24" x2="12.7" y2="12.7" width="0.4064" layer="1"/>
+<wire x1="12.7" y1="12.7" x2="10.16" y2="12.7" width="0.4064" layer="1"/>
 </signal>
 <signal name="GND">

Commit message: update
Parts:
- moved SV2 7.18 mm to (8.89, 25.4)
- moved SV1 2.84 mm to (8.89, 8.89)
Routing:
- net N$3: track 38.0 -> 24.4 mm
- net N$1: track 33.3 -> 21.9 mm
- net N$6: track 18.8 -> 13.2 mm
- net N$5: track 24.7 -> 29.8 mm
- net N$4: track 19.9 -> 16.8 mm
- net N$2: track 28.2 -> 27.0 mm
Other:
- board size 24.1 x 40.3 mm -> 17.8 x 35.2 mm
Changed lines of the file:
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@@
 <board>
 <plain>
-<wire x1="0" y1="0" x2="24.11" y2="0" width="0" layer="20"/>
-<wire x1="24.11" y1="0" x2="24.11" y2="40.31" width="0" layer="20"/>
-<wire x1="24.11" y1="40.31" x2="0" y2="40.31" width="0" layer="20"/>
-<wire x1="0" y1="40.31" x2="0" y2="0" width="0" layer="20"/>
-<hole x="17.78" y="7.62" drill="1.3"/>
-<hole x="5.08" y="35.56" drill="1.3"/>
-<dimension x1="24.11" y1="40.31" x2="27.94" y2="0" x3="26.67" y3="20.155" textsize="1.778" layer="25" dtype="vertical"/>
-<dimension x1="0" y1="40.31" x2="24.13" y2="43.18" x3="12.065" y3="41.91" textsize="1.778" layer="25" dtype="horizontal"/>
+<wire x1="0" y1="0" x2="17.76" y2="0" width="0" layer="20"/>
+<wire x1="17.76" y1="0" x2="17.76" y2="35.23" width="0" layer="20"/>
+<wire x1="17.76" y1="35.23" x2="0" y2="35.23" width="0" layer="20"/>
+<wire x1="0" y1="35.23" x2="0" y2="0" width="0" layer="20"/>
+<dimension x1="17.76" y1="0" x2="17.76" y2="35.23" x3="22.86" y3="17.615" textsize="1.778" layer="20"/>
+<dimension x1="0" y1="0" x2="17.76" y2="0" x3="8.88" y3="-3.81" textsize="1.778" layer="20"/>
 </plain>
 <attributes>
@@
 <param name="rvMicroViaOuter" value="0.25"/>
 <param name="rvMicroViaInner" value="0.25"/>
-<param name="rlMinPadTop" value="10mil"/>
+<param name="rlMinPadTop" value="17mil"/>
 <param name="rlMaxPadTop" value="20mil"/>
 <param name="rlMinPadInner" value="10mil"/>
@@
 </autorouter>
 <elements>
-<element name="SV1" library="con-lstb" package="MA03-2" value="" x="7.62" y="11.43">
-<attribute name="OC_NEWARK" value="unknown" x="7.62" y="11.43" size="1.778" layer="27" display="off"/>
-<attribute name="MPN" value="" x="7.62" y="11.43" size="1.778" layer="27" display="off"/>
-<attribute name="MF" value="" x="7.62" y="11.43" size="1.778" layer="27" display="off"/>
-<attribute name="OC_FARNELL" value="unknown" x="7.62" y="11.43" size="1.778" layer="27" display="off"/>
+<element name="SV1" library="con-lstb" package="MA03-2" value="" x="8.89" y="8.89">
+<attribute name="OC_NEWARK" value="unknown" x="8.89" y="8.89" size="1.778" layer="27" display="off"/>
+<attribute name="MPN" value="" x="8.89" y="8.89" size="1.778" layer="27" display="off"/>
+<attribute name="MF" value="" x="8.89" y="8.89" size="1.778" layer="27" display="off"/>
+<attribute name="OC_FARNELL" value="unknown" x="8.89" y="8.89" size="1.778" layer="27" display="off"/>
 </element>
-<element name="SV2" library="con-lstb" package="MA03-2" value="" x="13.97" y="30.48" rot="R270">
-<attribute name="OC_NEWARK" value="unknown" x="13.97" y="30.48" size="1.778" layer="27" rot="R270" display="off"/>
-<attribute name="MPN" value="" x="13.97" y="30.48" size="1.778" layer="27" rot="R270" display="off"/>
-<attribute name="MF" value="" x="13.97" y="30.48" size="1.778" layer="27" rot="R270" display="off"/>
-<attribute name="OC_FARNELL" value="unknown" x="13.97" y="30.48" size="1.778" layer="27" rot="R270" display="off"/>
+<element name="SV2" library="con-lstb" package="MA03-2" value="" x="8.89" y="25.4" rot="R270">
+<attribute name="OC_NEWARK" value="unknown" x="8.89" y="25.4" size="1.778" layer="27" rot="R270" display="off"/>
+<attribute name="MPN" value="" x="8.89" y="25.4" size="1.778" layer="27" rot="R270" display="off"/>
+<attribute name="MF" value="" x="8.89" y="25.4" size="1.778" layer="27" rot="R270" display="off"/>
+<attribute name="OC_FARNELL" value="unknown" x="8.89" y="25.4" size="1.778" layer="27" rot="R270" display="off"/>
 </element>
 </elements>
@@
 <contactref element="SV2" pad="2"/>
 <contactref element="SV1" pad="2"/>
-<wire x1="5.08" y1="12.7" x2="5.08" y2="31.75" width="0.4064" layer="1"/>
-<wire x1="5.08" y1="31.75" x2="8.89" y2="35.56" width="0.4064" layer="1"/>
-<wire x1="8.89" y1="35.56" x2="15.24" y2="35.56" width="0.4064" layer="1"/>
-<wire x1="15.24" y1="35.56" x2="15.24" y2="33.02" width="0.4064" layer="1"/>
+<wire x1="10.16" y1="27.94" x2="8.89" y2="26.67" width="0.6096" layer="1"/>
+<wire x1="6.35" y1="24.13" x2="5.08" y2="22.86" width="0.6096" layer="1"/>
+<wire x1="5.08" y1="22.86" x2="5.08" y2="11.43" width="0.6096" layer="1"/>
+<wire x1="5.08" y1="11.43" x2="6.35" y2="10.16" width="0.6096" layer="1"/>
+<wire x1="8.89" y1="26.67" x2="8.89" y2="24.13" width="0.6096" layer="1"/>
+<wire x1="8.89" y1="24.13" x2="6.35" y2="24.13" width="0.6096" layer="1"/>
 </signal>
 <signal name="N$2">
 <contactref element="SV2" pad="1"/>
 <contactref element="SV1" pad="1"/>
-<wire x1="5.08" y1="10.16" x2="6.35" y2="11.43" width="0.4064" layer="1"/>
-<wire x1="6.35" y1="11.43" x2="6.35" y2="30.48" width="0.4064" layer="1"/>
-<wire x1="6.35" y1="30.48" x2="8.89" y2="33.02" width="0.4064" layer="1"/>
-<wire x1="8.89" y1="33.02" x2="12.7" y2="33.02" width="0.4064" layer="1"/>
+<wire x1="7.62" y1="27.94" x2="5.08" y2="27.94" width="0.6096" layer="1"/>
+<wire x1="5.08" y1="27.94" x2="2.54" y2="25.4" width="0.6096" layer="1"/>
+<wire x1="2.54" y1="25.4" x2="2.54" y2="8.89" width="0.6096" layer="1"/>
+<wire x1="2.54" y1="8.89" x2="3.81" y2="7.62" width="0.6096" layer="1"/>
+<wire x1="3.81" y1="7.62" x2="6.35" y2="7.62" width="0.6096" layer="1"/>
 </signal>
 <signal name="N$3">
 <contactref element="SV2" pad="3"/>
 <contactref element="SV1" pad="3"/>
-<wire x1="7.62" y1="10.16" x2="10.16" y2="7.62" width="0.4064" layer="1"/>
-<wire x1="10.16" y1="7.62" x2="12.7" y2="7.62" width="0.4064" layer="1"/>
-<wire x1="12.7" y1="7.62" x2="17.78" y2="12.7" width="0.4064" layer="1"/>
-<wire x1="17.78" y1="12.7" x2="17.78" y2="31.75" width="0.4064" layer="1"/>
-<wire x1="17.78" y1="31.75" x2="13.97" y2="31.75" width="0.4064" layer="1"/>
-<wire x1="13.97" y1="31.75" x2="12.7" y2="30.48" width="0.4064" layer="1"/>
+<wire x1="7.62" y1="25.4" x2="5.08" y2="25.4" width="0.6096" layer="1"/>
+<wire x1="5.08" y1="25.4" x2="3.81" y2="24.13" width="0.6096" layer="1"/>
+<wire x1="3.81" y1="24.13" x2="3.81" y2="10.16" width="0.6096" layer="1"/>
+<wire x1="3.81" y1="10.16" x2="5.08" y2="8.89" width="0.6096" layer="1"/>
+<wire x1="5.08" y1="8.89" x2="7.62" y2="8.89" width="0.6096" layer="1"/>
+<wire x1="7.62" y1="8.89" x2="8.89" y2="7.62" width="0.6096" layer="1"/>
 </signal>
 <signal name="N$4">
 <contactref element="SV2" pad="5"/>
 <contactref element="SV1" pad="5"/>
-<wire x1="10.16" y1="10.16" x2="8.89" y2="11.43" width="0.4064" layer="1"/>
-<wire x1="8.89" y1="11.43" x2="8.89" y2="13.97" width="0.4064" layer="1"/>
-<wire x1="8.89" y1="13.97" x2="12.7" y2="17.78" width="0.4064" layer="1"/>
-<wire x1="12.7" y1="17.78" x2="12.7" y2="27.94" width="0.4064" layer="1"/>
+<wire x1="7.62" y1="22.86" x2="7.62" y2="17.78" width="0.6096" layer="1"/>
+<wire x1="7.62" y1="17.78" x2="10.16" y2="15.24" width="0.6096" layer="1"/>
+<wire x1="10.16" y1="15.24" x2="10.16" y2="10.16" width="0.6096" layer="1"/>
+<wire x1="10.16" y1="10.16" x2="11.43" y2="8.89" width="0.6096" layer="1"/>
+<wire x1="11.43" y1="8.89" x2="11.43" y2="7.62" width="0.6096" layer="1"/>
 </signal>
 <signal name="N$5">
 <contactref element="SV2" pad="4"/>
 <contactref element="SV1" pad="4"/>
-<wire x1="7.62" y1="12.7" x2="7.62" y2="29.21" width="0.4064" layer="1"/>
-<wire x1="7.62" y1="29.21" x2="13.97" y2="29.21" width="0.4064" layer="1"/>
-<wire x1="13.97" y1="29.21" x2="15.24" y2="30.48" width="0.4064" layer="1"/>
+<wire x1="10.16" y1="25.4" x2="12.7" y2="22.86" width="0.6096" layer="1"/>
+<wire x1="12.7" y1="22.86" x2="12.7" y2="12.7" width="0.6096" layer="1"/>
+<wire x1="12.7" y1="12.7" x2="13.97" y2="11.43" width="0.6096" layer="1"/>
+<wire x1="13.97" y1="11.43" x2="13.97" y2="6.35" width="0.6096" layer="1"/>
+<wire x1="13.97" y1="6.35" x2="12.7" y2="5.08" width="0.6096" layer="1"/>
+<wire x1="12.7" y1="5.08" x2="11.43" y2="5.08" width="0.6096" layer="1"/>
+<wire x1="11.43" y1="5.08" x2="10.16" y2="6.35" width="0.6096" layer="1"/>
+<wire x1="10.16" y1="6.35" x2="10.16" y2="8.89" width="0.6096" layer="1"/>
+<wire x1="10.16" y1="8.89" x2="8.89" y2="10.16" width="0.6096" layer="1"/>
 </signal>
 <signal name="N$6">
 <contactref element="SV2" pad="6"/>
 <contactref element="SV1" pad="6"/>
-<wire x1="15.24" y1="27.94" x2="15.24" y2="15.24" width="0.4064" layer="1"/>
-<wire x1="15.24" y1="15.24" x2="12.7" y2="12.7" width="0.4064" layer="1"/>
-<wire x1="12.7" y1="12.7" x2="10.16" y2="12.7" width="0.4064" layer="1"/>
+<wire x1="10.16" y1="22.86" x2="10.16" y2="17.78" width="0.6096" layer="1"/>
+<wire x1="10.16" y1="17.78" x2="11.43" y2="16.51" width="0.6096" layer="1"/>
+<wire x1="11.43" y1="16.51" x2="11.43" y2="10.16" width="0.6096" layer="1"/>
 </signal>
 <signal name="GND">
 <polygon width="0.4064" layer="1">
-<vertex x="1.27" y="39.37"/>
+<vertex x="1.27" y="34.29"/>
 <vertex x="1.27" y="1.27"/>
-<vertex x="22.86" y="1.27"/>
-<vertex x="22.86" y="39.37"/>
+<vertex x="16.51" y="1.27"/>
+<vertex x="16.51" y="34.29"/>
 </polygon>
 </signal>
